File: Hardware/TP540xEVM.kicad_sch (KiCad schematic)
At the start: 11 parts, among them U1 TPS5403

Commit message: ...
Parts:
- added J1: Input, TerminalBlock_4Ucon:TerminalBlock_4Ucon_1x02_P3.50mm_Horizontal, symbol Connector:Conn_01x02_Male
- added J2: Output, TerminalBlock_4Ucon:TerminalBlock_4Ucon_1x02_P3.50mm_Horizontal, symbol Connector:Conn_01x02_Male
- C2, C3: value 220uF -> 330uF; footprint Capacitor_SMD:CP_Elec_3x5.3 -> Capacitor_SMD:CP_Elec_8x10; LCSC (none) -> C178599
- D1: value D_Schottky -> DSK24; footprint Diode_SMD:D_SMA -> Diode_SMD:D_SOD-123; LCSC (none) -> C908229
Connections:
- net GND: now also J1.2 (Pin_2), J2.1 (Pin_1)
- net Vin: now also J1.1 (Pin_1)
- net Vout: now also J2.2 (Pin_2)
Changed lines of the file:
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@@
     (stroke (width 0) (type default) (color 0 0 0 0))
+  )
+  (global_label "Vout" (shape input) (at 199.39 67.31 90) (fields_autoplaced)
+    (effects (font (size 1.27 1.27)) (justify left))
+    (property "Intersheet References" "${INTERSHEET_REFS}" (id 0) (at 199.3106 60.7845 90)
+      (effects (font (size 1.27 1.27)) (justify left) hide)
+    )
+  )
+  (global_label "Vin" (shape input) (at 105.41 67.31 90) (fields_autoplaced)
+    (effects (font (size 1.27 1.27)) (justify left))
+    (property "Intersheet References" "${INTERSHEET_REFS}" (id 0) (at 105.3306 62.0545 90)
+      (effects (font (size 1.27 1.27)) (justify left) hide)
+    )
   )
   (global_label "Vout" (shape input) (at 195.58 93.98 90) (fields_autoplaced)
@@
     (pin "2")
   )
+  (symbol (lib_id "power:GND") (at 199.39 69.85 0) (unit 1)
+    (in_bom yes) (on_board yes) (fields_autoplaced)
+    (property "Reference" "#PWR0109" (id 0) (at 199.39 76.2 0)
+      (effects (font (size 1.27 1.27)) hide)
+    )
+    (property "Value" "GND" (id 1) (at 199.39 74.93 0))
+    (property "Footprint" "" (id 2) (at 199.39 69.85 0)
+      (effects (font (size 1.27 1.27)) hide)
+    )
+    (property "Datasheet" "" (id 3) (at 199.39 69.85 0)
+      (effects (font (size 1.27 1.27)) hide)
+    )
+    (pin "1")
+  )
   (symbol (lib_id "power:GND") (at 105.41 116.84 0) (unit 1)
     (in_bom yes) (on_board yes) (fields_autoplaced)
@@
       (effects (font (size 1.27 1.27)) (justify left))
     )
-    (property "Value" "220uF" (id 1) (at 80.01 93.0909 0)
-      (effects (font (size 1.27 1.27)) (justify left))
-    )
-    (property "Footprint" "Capacitor_SMD:CP_Elec_3x5.3" (id 2) (at 77.1652 96.52 0)
+    (property "Value" "330uF" (id 1) (at 80.01 93.0909 0)
+      (effects (font (size 1.27 1.27)) (justify left))
+    )
+    (property "Footprint" "Capacitor_SMD:CP_Elec_8x10" (id 2) (at 77.1652 96.52 0)
       (effects (font (size 1.27 1.27)) hide)
     )
@@
       (effects (font (size 1.27 1.27)) hide)
     )
+    (property "LCSC" "C178599" (id 4) (at 76.2 92.71 0)
+      (effects (font (size 1.27 1.27)) hide)
+    )
     (pin "1")
     (pin "2")
@@
       (effects (font (size 1.27 1.27)) (justify left))
     )
-    (property "Value" "D_Schottky" (id 1) (at 166.37 98.7424 90)
-      (effects (font (size 1.27 1.27)) (justify left))
-    )
-    (property "Footprint" "Diode_SMD:D_SMA" (id 2) (at 163.83 97.79 0)
+    (property "Value" "DSK24" (id 1) (at 166.37 98.7424 90)
+      (effects (font (size 1.27 1.27)) (justify left))
+    )
+    (property "Footprint" "Diode_SMD:D_SOD-123" (id 2) (at 163.83 97.79 0)
       (effects (font (size 1.27 1.27)) hide)
     )
@@
       (effects (font (size 1.27 1.27)) hide)
     )
+    (property "LCSC" "C908229" (id 4) (at 163.83 97.79 90)
+      (effects (font (size 1.27 1.27)) hide)
+    )
     (pin "1")
     (pin "2")
@@
     (pin "2")
   )
+  (symbol (lib_id "power:GND") (at 105.41 69.85 0) (unit 1)
+    (in_bom yes) (on_board yes) (fields_autoplaced)
+    (property "Reference" "#PWR0108" (id 0) (at 105.41 76.2 0)
+      (effects (font (size 1.27 1.27)) hide)
+    )
+    (property "Value" "GND" (id 1) (at 105.41 74.93 0))
+    (property "Footprint" "" (id 2) (at 105.41 69.85 0)
+      (effects (font (size 1.27 1.27)) hide)
+    )
+    (property "Datasheet" "" (id 3) (at 105.41 69.85 0)
+      (effects (font (size 1.27 1.27)) hide)
+    )
+    (pin "1")
+  )
   (symbol (lib_id "Device:C_Polarized") (at 201.93 97.79 0) (unit 1)
     (in_bom yes) (on_board yes) (fields_autoplaced)
@@
       (effects (font (size 1.27 1.27)) (justify left))
     )
-    (property "Value" "220uF" (id 1) (at 205.74 98.1709 0)
-      (effects (font (size 1.27 1.27)) (justify left))
-    )
-    (property "Footprint" "Capacitor_SMD:CP_Elec_3x5.3" (id 2) (at 202.8952 101.6 0)
+    (property "Value" "330uF" (id 1) (at 205.74 98.1709 0)
+      (effects (font (size 1.27 1.27)) (justify left))
+    )
+    (property "Footprint" "Capacitor_SMD:CP_Elec_8x10" (id 2) (at 202.8952 101.6 0)
       (effects (font (size 1.27 1.27)) hide)
     )
     (property "Datasheet" "~" (id 3) (at 201.93 97.79 0)
+      (effects (font (size 1.27 1.27)) hide)
+    )
+    (property "LCSC" "C178599" (id 4) (at 201.93 97.79 0)
       (effects (font (size 1.27 1.27)) hide)
     )
@@
     (pin "1")
   )
+  (symbol (lib_id "Connector:Conn_01x02_Male") (at 100.33 67.31 0) (unit 1)
+    (in_bom yes) (on_board yes) (fields_autoplaced)
+    (property "Reference" "J1" (id 0) (at 100.965 62.23 0))
+    (property "Value" "Input" (id 1) (at 100.965 64.77 0))
+    (property "Footprint" "TerminalBlock_4Ucon:TerminalBlock_4Ucon_1x02_P3.50mm_Horizontal" (id 2) (at 100.33 67.31 0)
+      (effects (font (size 1.27 1.27)) hide)
+    )
+    (property "Datasheet" "~" (id 3) (at 100.33 67.31 0)
+      (effects (font (size 1.27 1.27)) hide)
+    )
+    (property "LCSC" "C784940" (id 4) (at 100.33 67.31 0)
+      (effects (font (size 1.27 1.27)) hide)
+    )
+    (pin "1")
+    (pin "2")
+  )
   (symbol (lib_id "power:GND") (at 87.63 107.95 0) (unit 1)
     (in_bom yes) (on_board yes) (fields_autoplaced)
@@
     )
     (pin "1")
+  )
+  (symbol (lib_id "Connector:Conn_01x02_Male") (at 194.31 69.85 0) (mirror x) (unit 1)
+    (in_bom yes) (on_board yes) (fields_autoplaced)
+    (property "Reference" "J2" (id 0) (at 193.04 67.3099 0)
+      (effects (font (size 1.27 1.27)) (justify right))
+    )
+    (property "Value" "Output" (id 1) (at 193.04 69.8499 0)
+      (effects (font (size 1.27 1.27)) (justify right))
+    )
+    (property "Footprint" "TerminalBlock_4Ucon:TerminalBlock_4Ucon_1x02_P3.50mm_Horizontal" (id 2) (at 194.31 69.85 0)
+      (effects (font (size 1.27 1.27)) hide)
+    )
+    (property "Datasheet" "~" (id 3) (at 194.31 69.85 0)
+      (effects (font (size 1.27 1.27)) hide)
+    )
+    (property "LCSC" "C784940" (id 4) (at 194.31 69.85 0)
+      (effects (font (size 1.27 1.27)) hide)
+    )
+    (pin "1")
+    (pin "2")
   )
   (symbol (lib_id "Device:C") (at 99.06 111.76 0) (unit 1)
@@
       (reference "#PWR0107") (unit 1) (value "GND") (footprint "")
     )
+    (path "/7fabf717-72b8-47c5-a9b7-190c0b4434a3"
+      (reference "#PWR0108") (unit 1) (value "GND") (footprint "")
+    )
+    (path "/49028326-7daa-445b-a931-57e602dabcb3"
+      (reference "#PWR0109") (unit 1) (value "GND") (footprint "")
+    )
     (path "/6eb6f4bc-ffe4-4e21-b5ae-ab6bf1df2410"
       (reference "C1") (unit 1) (value "0.1uF") (footprint "Capacitor_SMD:C_0603_1608Metric_Pad1.08x0.95mm_HandSolder")
     )
     (path "/65f6c523-f6b8-4923-a049-e8aaab3c528c"
-      (reference "C2") (unit 1) (value "220uF") (footprint "Capacitor_SMD:CP_Elec_3x5.3")
+      (reference "C2") (unit 1) (value "330uF") (footprint "Capacitor_SMD:CP_Elec_8x10")
     )
     (path "/8df82a26-e047-4f1c-9c3a-25d9d3df83bc"
-      (reference "C3") (unit 1) (value "220uF") (footprint "Capacitor_SMD:CP_Elec_3x5.3")
+      (reference "C3") (unit 1) (value "330uF") (footprint "Capacitor_SMD:CP_Elec_8x10")
     )
     (path "/6dabc724-b29c-42b8-be78-338f0a1680c7"
@@
     )
     (path "/721841bf-d919-4166-a5d1-28c1350f4278"
-      (reference "D1") (unit 1) (value "D_Schottky") (footprint "Diode_SMD:D_SMA")
+      (reference "D1") (unit 1) (value "DSK24") (footprint "Diode_SMD:D_SOD-123")
+    )
+    (path "/a1685dea-bc86-475b-ba60-d8aa7ab025ac"
+      (reference "J1") (unit 1) (value "Input") (footprint "TerminalBlock_4Ucon:TerminalBlock_4Ucon_1x02_P3.50mm_Horizontal")
+    )
+    (path "/b72be724-b1d9-412e-87fa-4a31db0be06e"
+      (reference "J2") (unit 1) (value "Output") (footprint "TerminalBlock_4Ucon:TerminalBlock_4Ucon_1x02_P3.50mm_Horizontal")
     )
     (path "/479f3f0b-5f70-458d-a591-f099cd39a0d2"
