File: Hardware/TP540xEVM.kicad_pcb (KiCad board)
At the start: 2 copper layers, 27.9 x 20.3 mm, 11 parts, among them U1 TPS5403

Commit message: ...
Parts:
- added J1: Input, TerminalBlock_4Ucon:TerminalBlock_4Ucon_1x02_P3.50mm_Horizontal, F.Cu at (86.7, 96.5)
- added J2: Output, TerminalBlock_4Ucon:TerminalBlock_4Ucon_1x02_P3.50mm_Horizontal, F.Cu at (113.3, 100.0)
- added REF**: Mount, Tinker:Mount, F.Cu at (114.8, 109.6)
- added REF**: Mount, Tinker:Mount, F.Cu at (85.2, 90.4)
- added REF**: Mount, Tinker:Mount, F.Cu at (85.2, 109.6)
- added REF**: DagNabbit, Tinker:DagNabbit, F.Cu at (99.9, 104.0)
- added REF**: Mount, Tinker:Mount, F.Cu at (114.8, 90.4)
- C2, C3: value 220uF -> 330uF; footprint Capacitor_SMD:CP_Elec_3x5.3 -> Capacitor_SMD:CP_Elec_8x10
- D1: value D_Schottky -> DSK24; footprint Diode_SMD:D_SMA -> Diode_SMD:D_SOD-123
- moved D1 52.6 mm to (104.5, 89.0), turned to 0 degrees
- moved C3 51.7 mm to (106.7, 107.3)
- moved C1 46.2 mm to (96.9, 89.1)
- moved C4 46.2 mm to (96.9, 98.0)
- moved R2 46.2 mm to (99.4, 98.0)
- moved U1 46.2 mm to (96.9, 92.9)
- moved C5 46.2 mm to (94.3, 98.0)
- moved C6 46.2 mm to (101.9, 98.0)
- moved R1 46.2 mm to (91.8, 98.0)
- moved L1 45.4 mm to (105.1, 91.7)
- moved C2 42.3 mm to (93.3, 107.3)
Routing:
- net Vin: track 13.7 -> 21.4 mm
- net Vout: track 19.7 -> 23.7 mm, vias 2 -> 1
- net Net-(R1-Pad1): track 4.83 -> 5.39 mm
- net Net-(C1-Pad2): track 13.5 -> 13.0 mm
Other:
- board size 27.9 x 20.3 mm -> 36 x 25.7 mm
- board text added: "+"
- board text added: "18.415 x 12.680"
- board text added: "G"
- board text added: "IN"
- board text added: "OUT"
- board text removed: "21.590 x 12.700"

Commit message: ...
Parts:
- moved D1 2.24 mm to (102.2, 89.0)
- moved REF** 0.51 mm to (100.0, 103.5)
Routing:
- net Net-(C1-Pad2): track 13.0 -> 11.2 mm
Other:
- board text added: "18.0 x 12.2"
- board text removed: "18.415 x 12.680"
Changed lines of the file:
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@@
   (net 9 "Net-(R1-Pad1)")
   (footprint "Diode_SMD:D_SOD-123" (layer "F.Cu")
-    (at 104.4767 89)
+    (at 102.235 89)
     (descr "SOD-123")
     (tags "SOD-123")
@@
   )
   (footprint "Tinker:DagNabbit" (layer "F.Cu")
-    (at 99.9 104 180)
+    (at 100 103.5 180)
     (attr smd board_only)
     (fp_text reference "REF**" (at 0 -8.08 180 unlocked) (layer "F.SilkS") hide
@@
     (pad "" np_thru_hole circle (at 0 0) (size 3.2 3.2) (drill 3.2) (layers *.Mask))
   )
-  (gr_line (start 109.5 100.5) (end 109.5 87.82) (layer "F.SilkS") (width 0.15))
-  (gr_line (start 109.5 87.82) (end 90.5 87.82) (layer "F.SilkS") (width 0.15))
-  (gr_line (start 90.5 87.82) (end 90.5067 100.5) (layer "F.SilkS") (width 0.15))
-  (gr_line (start 90.5067 100.5) (end 109.5 100.5) (layer "F.SilkS") (width 0.15))
+  (gr_line (start 109 100) (end 109 87.8) (layer "F.SilkS") (width 0.15))
+  (gr_line (start 109 87.8) (end 91 87.8) (layer "F.SilkS") (width 0.15))
+  (gr_line (start 91 87.8) (end 91 100) (layer "F.SilkS") (width 0.15))
+  (gr_line (start 91 100) (end 109 100) (layer "F.SilkS") (width 0.15))
   (gr_line (start 118 109.6958) (end 118 90.36) (layer "Edge.Cuts") (width 0.1))
   (gr_line (start 85.175 112.879936) (end 114.825 112.8708) (layer "Edge.Cuts") (width 0.1))
@@
     (effects (font (size 1 1) (thickness 0.15)))
   )
-  (gr_text "18.415\nx\n12.680" (at 107.0167 98.615) (layer "F.SilkS")
+  (gr_text "18.0 x 12.2" (at 106 99.5) (layer "F.SilkS")
     (effects (font (size 0.6 0.6) (thickness 0.15)))
   )
@@
   (segment (start 95.9942 89.09) (end 95.9942 89.3825) (width 0.25) (layer "F.Cu") (net 1))
   (segment (start 95.9942 89.3825) (end 94.3817 90.995) (width 0.25) (layer "F.Cu") (net 1))
-  (segment (start 100.8317 90.995) (end 102.8267 89) (width 0.6) (layer "F.Cu") (net 2))
   (segment (start 99.3317 90.995) (end 104.4067 90.995) (width 0.6) (layer "F.Cu") (net 2))
-  (segment (start 99.3317 90.995) (end 100.8317 90.995) (width 0.6) (layer "F.Cu") (net 2))
   (segment (start 104.4067 90.995) (end 105.1117 91.7) (width 0.6) (layer "F.Cu") (net 2))
+  (segment (start 100.585 89.7417) (end 100.585 89) (width 0.6) (layer "F.Cu") (net 2))
   (segment (start 97.7192 89.3825) (end 99.3317 90.995) (width 0.25) (layer "F.Cu") (net 2))
   (segment (start 97.7192 89.09) (end 97.7192 89.3825) (width 0.25) (layer "F.Cu") (net 2))
+  (segment (start 99.3317 90.995) (end 100.585 89.7417) (width 0.6) (layer "F.Cu") (net 2))
   (segment (start 89.8717 100.06) (end 92.71 102.8983) (width 0.6) (layer "F.Cu") (net 3))
   (segment (start 86.6967 94.805) (end 86.6967 96.5167) (width 0.6) (layer "F.Cu") (net 3))
