File: Standalone Hardware/TP540xEVM.kicad_pcb (KiCad board)
At the start: 2 copper layers, 36 x 25.7 mm, 18 parts, among them J1 Input, J2 Output, U1 TPS5403

Commit message: ...
Parts:
- moved L1 4.07 mm to (104.7, 95.7)
- moved D1 2.86 mm to (104.7, 90.4)
- moved R1 2.55 mm to (94.0, 99.2)
- moved C6 1.98 mm to (100.4, 99.2), turned to 90 degrees
- moved C5 1.79 mm to (95.6, 99.2)
- moved C1 1.55 mm to (96.9, 90.6)
- moved R2 1.38 mm to (98.8, 99.2)
- moved REF** 1.30 mm to (99.9, 104.8)
- moved C4 1.29 mm to (97.2, 99.2)
- moved U1 1.24 mm to (96.9, 94.1)
- moved C2 0.32 mm to (93.0, 107.2)
- moved C3 0.32 mm to (107.0, 107.2)
Routing:
- net Net-(C6-Pad1): track 3.28 -> 1.62 mm
- net Vin: track 21.4 -> 19.9 mm
- net Net-(R1-Pad1): track 5.39 -> 5.98 mm
- net Vout: track 23.7 -> 23.1 mm, vias 1 -> 0
- net Net-(C4-Pad1): track 8.64 -> 8.77 mm, vias 0 -> 2
Other:
- board text added: "16.0 x 12.0"
- board text added: "S. A. Miller 2024"
- board text added: "TPS540x Breakout"
- board text removed: "18.0 x 12.2"
