File: Standalone Hardware/TP540xEVM.kicad_pcb (KiCad board)
At the start: 2 copper layers, 36 x 25.7 mm, 18 parts, among them J1 Input, J2 Output, U1 TPS5403

Commit message: w00t...SMD inductor
Parts:
- L1: footprint Inductor_THT:L_Radial_D6.0mm_P4.00mm -> Tinker:IND-SMD_L7.1-W6.6
- moved L1 0.33 mm to (104.4, 95.8)
Changed lines of the file:
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@@
     )
   )
-  (footprint "Inductor_THT:L_Radial_D6.0mm_P4.00mm" (layer "F.Cu")
-    (at 104.7 95.745 -90)
-    (descr "Inductor, Radial series, Radial, pin pitch=4.00mm, , diameter=6.0mm, http://www.abracon.com/Magnetics/radial/AIUR-07.pdf")
-    (tags "Inductor Radial series Radial pin pitch 4.00mm  diameter 6.0mm")
+  (footprint "Tinker:IND-SMD_L7.1-W6.6" (layer "F.Cu")
+    (at 104.372882 95.753077 -90)
     (property "Sheetfile" "TP540xEVM.kicad_sch")
     (property "Sheetname" "")
-    (attr through_hole)
-    (fp_text reference "L1" (at 3.29 2.265) (layer "F.SilkS")
+    (attr smd)
+    (fp_text reference "L1" (at 3.941923 2.57) (layer "F.SilkS")
       (effects (font (size 0.6 0.6) (thickness 0.15)))
     )
-    (fp_text value "L_Ferrite" (at 0 5.08 90) (layer "F.Fab")
+    (fp_text value "L_Ferrite" (at 0 4 -90) (layer "F.Fab")
       (effects (font (size 1 1) (thickness 0.15)))
     )
-    (fp_text user "${REFERENCE}" (at 0 -5.08 90) (layer "F.Fab")
+    (fp_text user "${REFERENCE}" (at 0 0 -90) (layer "F.Fab")
       (effects (font (size 1 1) (thickness 0.15)))
     )
-    (fp_arc (start 2.85426 1.26) (mid 0 3.12) (end -2.85426 1.26) (layer "F.SilkS") (width 0.12))
-    (fp_arc (start -2.85426 -1.26) (mid 0 -3.12) (end 2.85426 -1.26) (layer "F.SilkS") (width 0.12))
-    (fp_circle (center 0 0) (end 4 0) (layer "F.CrtYd") (width 0.05) (fill none))
-    (fp_circle (center 0 0) (end 3 0) (layer "F.Fab") (width 0.1) (fill none))
-    (pad "1" thru_hole circle (at -2.5 0 270) (size 2 2) (drill 1) (layers *.Cu *.Mask)
+    (fp_line (start -3.3 3.3) (end 3.3 3.3) (layer "F.SilkS") (width 0.15))
+    (fp_line (start -3.3 1.84) (end -3.3 3.3) (layer "F.SilkS") (width 0.15))
+    (fp_line (start 3.3 -3.3) (end -3.3 -3.3) (layer "F.SilkS") (width 0.15))
+    (fp_line (start -3.3 -3.3) (end -3.3 -1.84) (layer "F.SilkS") (width 0.15))
+    (fp_line (start 3.3 -1.84) (end 3.3 -3.3) (layer "F.SilkS") (width 0.15))
+    (fp_line (start 3.3 3.3) (end 3.3 1.84) (layer "F.SilkS") (width 0.15))
+    (fp_circle (center -3.55 3.3) (end -3.52 3.3) (layer "F.Fab") (width 0.06) (fill none))
+    (pad "1" smd rect (at -2.91 0 270) (size 2.15 3.32) (layers "F.Cu" "F.Paste" "F.Mask")
       (net 2 "Net-(C1-Pad2)") (pinfunction "1") (pintype "passive"))
-    (pad "2" thru_hole circle (at 2.5 0 270) (size 2 2) (drill 1) (layers *.Cu *.Mask)
+    (pad "2" smd rect (at 2.91 0 270) (size 2.15 3.32) (layers "F.Cu" "F.Paste" "F.Mask")
       (net 5 "Vout") (pinfunction "2") (pintype "passive"))
-    (model "${KICAD6_3DMODEL_DIR}/Inductor_THT.3dshapes/L_Radial_D6.0mm_P4.00mm.wrl"
-      (offset (xyz -2 0 0))
+    (model "/home/tinker/Documents/LCSC-KiCAD/.3dshapes/IND-SMD_L6.6-W7.1-H3.0.wrl"
+      (offset (xyz 0.11 0 0))
       (scale (xyz 1 1 1))
       (rotate (xyz 0 0 0))
