File: Standalone Hardware/TP540xEVM.kicad_sch (KiCad schematic)
At the start: 13 parts, among them J1 Input, J2 Output, U1 TPS5403

Commit message: ...
Parts:
- C1, C4, C5, C6: footprint Capacitor_SMD:C_0603_1608Metric_Pad1.08x0.95mm_HandSolder -> Capacitor_SMD:C_0603_1608Metric
- R1, R2: footprint Resistor_SMD:R_0603_1608Metric_Pad0.98x0.95mm_HandSolder -> Resistor_SMD:R_0603_1608Metric
Changed lines of the file:
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@@
       (effects (font (size 1.27 1.27)) (justify left))
     )
-    (property "Footprint" "Capacitor_SMD:C_0603_1608Metric_Pad1.08x0.95mm_HandSolder" (id 2) (at 111.4552 107.95 0)
+    (property "Footprint" "Capacitor_SMD:C_0603_1608Metric" (id 2) (at 111.4552 107.95 0)
       (effects (font (size 1.27 1.27)) hide)
     )
@@
       (effects (font (size 1.27 1.27)) (justify left))
     )
-    (property "Footprint" "Capacitor_SMD:C_0603_1608Metric_Pad1.08x0.95mm_HandSolder" (id 2) (at 164.7952 93.98 0)
+    (property "Footprint" "Capacitor_SMD:C_0603_1608Metric" (id 2) (at 164.7952 93.98 0)
       (effects (font (size 1.27 1.27)) hide)
     )
@@
       (effects (font (size 1.27 1.27)) (justify left))
     )
-    (property "Footprint" "Resistor_SMD:R_0603_1608Metric_Pad0.98x0.95mm_HandSolder" (id 2) (at 97.282 104.14 90)
+    (property "Footprint" "Resistor_SMD:R_0603_1608Metric" (id 2) (at 97.282 104.14 90)
       (effects (font (size 1.27 1.27)) hide)
     )
@@
       (effects (font (size 1.27 1.27)) (justify left))
     )
-    (property "Footprint" "Resistor_SMD:R_0603_1608Metric_Pad0.98x0.95mm_HandSolder" (id 2) (at 85.852 104.14 90)
+    (property "Footprint" "Resistor_SMD:R_0603_1608Metric" (id 2) (at 85.852 104.14 90)
       (effects (font (size 1.27 1.27)) hide)
     )
@@
       (effects (font (size 1.27 1.27)) (justify left))
     )
-    (property "Footprint" "Capacitor_SMD:C_0603_1608Metric_Pad1.08x0.95mm_HandSolder" (id 2) (at 100.0252 115.57 0)
+    (property "Footprint" "Capacitor_SMD:C_0603_1608Metric" (id 2) (at 100.0252 115.57 0)
       (effects (font (size 1.27 1.27)) hide)
     )
@@
       (effects (font (size 1.27 1.27)) (justify left))
     )
-    (property "Footprint" "Capacitor_SMD:C_0603_1608Metric_Pad1.08x0.95mm_HandSolder" (id 2) (at 125.4252 107.95 0)
+    (property "Footprint" "Capacitor_SMD:C_0603_1608Metric" (id 2) (at 125.4252 107.95 0)
       (effects (font (size 1.27 1.27)) hide)
     )
@@
     )
     (path "/6eb6f4bc-ffe4-4e21-b5ae-ab6bf1df2410"
-      (reference "C1") (unit 1) (value "0.1uF") (footprint "Capacitor_SMD:C_0603_1608Metric_Pad1.08x0.95mm_HandSolder")
+      (reference "C1") (unit 1) (value "0.1uF") (footprint "Capacitor_SMD:C_0603_1608Metric")
     )
     (path "/65f6c523-f6b8-4923-a049-e8aaab3c528c"
@@
     )
     (path "/6dabc724-b29c-42b8-be78-338f0a1680c7"
-      (reference "C4") (unit 1) (value "100pF") (footprint "Capacitor_SMD:C_0603_1608Metric_Pad1.08x0.95mm_HandSolder")
+      (reference "C4") (unit 1) (value "100pF") (footprint "Capacitor_SMD:C_0603_1608Metric")
     )
     (path "/e4e24123-44de-4b2c-9afe-5d69a05b67dc"
-      (reference "C5") (unit 1) (value "10nF") (footprint "Capacitor_SMD:C_0603_1608Metric_Pad1.08x0.95mm_HandSolder")
+      (reference "C5") (unit 1) (value "10nF") (footprint "Capacitor_SMD:C_0603_1608Metric")
     )
     (path "/cf200e13-0d43-4df2-9437-994bbc4c68a0"
-      (reference "C6") (unit 1) (value "2.2nF") (footprint "Capacitor_SMD:C_0603_1608Metric_Pad1.08x0.95mm_HandSolder")
+      (reference "C6") (unit 1) (value "2.2nF") (footprint "Capacitor_SMD:C_0603_1608Metric")
     )
     (path "/721841bf-d919-4166-a5d1-28c1350f4278"
@@
     )
     (path "/794b9bb4-29b7-450a-bb76-0318a7f3d068"
-      (reference "R1") (unit 1) (value "100K") (footprint "Resistor_SMD:R_0603_1608Metric_Pad0.98x0.95mm_HandSolder")
+      (reference "R1") (unit 1) (value "100K") (footprint "Resistor_SMD:R_0603_1608Metric")
     )
     (path "/70e58dde-9be7-47a9-b0c9-c4f2a606fac0"
-      (reference "R2") (unit 1) (value "47K") (footprint "Resistor_SMD:R_0603_1608Metric_Pad0.98x0.95mm_HandSolder")
+      (reference "R2") (unit 1) (value "47K") (footprint "Resistor_SMD:R_0603_1608Metric")
     )
     (path "/ee4d7171-d495-4a95-b1d9-8b3f26e1c580"

Commit message: w00t...SMD inductor
Parts:
- L1: footprint Inductor_THT:L_Radial_D6.0mm_P4.00mm -> Tinker:IND-SMD_L7.1-W6.6; LCSC (none) -> C2983095
Changed lines of the file:
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@@
     (property "Reference" "L1" (id 0) (at 181.61 87.63 90))
     (property "Value" "L_Ferrite" (id 1) (at 181.61 90.17 90))
-    (property "Footprint" "Inductor_THT:L_Radial_D6.0mm_P4.00mm" (id 2) (at 181.61 93.98 0)
+    (property "Footprint" "Tinker:IND-SMD_L7.1-W6.6" (id 2) (at 181.61 93.98 0)
       (effects (font (size 1.27 1.27)) hide)
     )
     (property "Datasheet" "~" (id 3) (at 181.61 93.98 0)
+      (effects (font (size 1.27 1.27)) hide)
+    )
+    (property "LCSC" "C2983095" (id 4) (at 181.61 93.98 90)
       (effects (font (size 1.27 1.27)) hide)
     )
@@
     )
     (path "/479f3f0b-5f70-458d-a591-f099cd39a0d2"
-      (reference "L1") (unit 1) (value "L_Ferrite") (footprint "Inductor_THT:L_Radial_D6.0mm_P4.00mm")
+      (reference "L1") (unit 1) (value "L_Ferrite") (footprint "Tinker:IND-SMD_L7.1-W6.6")
     )
     (path "/794b9bb4-29b7-450a-bb76-0318a7f3d068"
