File: Standalone Hardware/TP540xSAL.kicad_pcb (KiCad board)
At the start: 2 copper layers, 36 x 25.7 mm, 18 parts, among them J1 Input, J2 Output, U1 TPS5403

Commit message: Some cleanup...
Parts:
- added G***: LOGO, Tinker:NerdMage, F.Cu at (110.5, 90.8)
