File: Standalone Hardware (carrier)/TP540xEVM.kicad_pcb (KiCad board)
At the start: 2 copper layers, 36 x 25.7 mm, 18 parts, among them J1 Input, J2 Output, U1 TPS5403

Commit message: ...
Parts:
- removed C1: 0.1uF, Capacitor_SMD:C_0603_1608Metric
- removed C4: 100pF, Capacitor_SMD:C_0603_1608Metric
- removed C5: 10nF, Capacitor_SMD:C_0603_1608Metric
- removed C6: 2.2nF, Capacitor_SMD:C_0603_1608Metric
- removed D1: DSK24, Diode_SMD:D_SOD-123
- removed L1: L_Ferrite, Inductor_THT:L_Radial_D6.0mm_P4.00mm
- removed R1: 100K, Resistor_SMD:R_0603_1608Metric
- removed R2: 47K, Resistor_SMD:R_0603_1608Metric
- removed U1: TPS5403, Package_SO:SOIC-8_3.9x4.9mm_P1.27mm
- added J3: MountPoint, Tinker:ConnPoint, F.Cu at (90.8, 90.2)
- added J4: MountPoint, Tinker:ConnPoint, F.Cu at (109.2, 90.2)
- added J5: MountPoint, Tinker:ConnPoint, F.Cu at (90.8, 99.2)
- added J6: MountPoint, Tinker:ConnPoint, F.Cu at (109.2, 99.2)
- moved J1 0.67 mm to (86.0, 96.5)
- moved J2 0.67 mm to (114.0, 100.0)
Routing:
- net Net-(C1-Pad2): track 11.5 -> 0.00 mm
- net Net-(C4-Pad1): track 8.95 -> 0.00 mm, vias 2 -> 0
- net Net-(R1-Pad1): track 5.46 -> 0.00 mm
- net Vin: track 19.9 -> 23.0 mm
- net Net-(C5-Pad1): track 2.34 -> 0.00 mm
- net Net-(C1-Pad1): track 2.28 -> 0.00 mm
- net Net-(C6-Pad1): track 1.55 -> 0.00 mm
- net GND: vias 10 -> 0
Other:
- board text removed: "16.0 x 11.0"
