File: Standalone Hardware (carrier)/TP540xMCB.kicad_pcb (KiCad board)
At the start: 2 copper layers, 36 x 25.7 mm, 22 parts, among them J1 Input, J2 Output, J3 MountPoint, J4 MountPoint, J5 MountPoint, J6 MountPoint, U1 TPS5403

Commit message: w00t...SMD inductor
Parts:
- removed C1: 0.1uF, Capacitor_SMD:C_0603_1608Metric
- removed C4: 100pF, Capacitor_SMD:C_0603_1608Metric
- removed C5: 10nF, Capacitor_SMD:C_0603_1608Metric
- removed C6: 2.2nF, Capacitor_SMD:C_0603_1608Metric
- removed D1: DSK24, Diode_SMD:D_SOD-123
- removed L1: L_Ferrite, Inductor_THT:L_Radial_D6.0mm_P4.00mm
- removed R1: 100K, Resistor_SMD:R_0603_1608Metric
- removed R2: 47K, Resistor_SMD:R_0603_1608Metric
- removed U1: TPS5403, Package_SO:SOIC-8_3.9x4.9mm_P1.27mm
- moved J5 0.14 mm to (90.8, 99.2)
Routing:
- net Vout: track 37.9 -> 23.0 mm
- net Net-(C1-Pad2): track 11.5 -> 0.00 mm
- net Net-(C4-Pad1): track 8.95 -> 0.00 mm, vias 2 -> 0
- net Net-(R1-Pad1): track 5.46 -> 0.00 mm
- net Vin: track 26.8 -> 23.0 mm
- net Net-(C5-Pad1): track 2.34 -> 0.00 mm
- net Net-(C1-Pad1): track 2.28 -> 0.00 mm
- net Net-(C6-Pad1): track 1.55 -> 0.00 mm
- net GND: vias 10 -> 0
Other:
- board text removed: "16.0 x 11.0"
