File: Standalone Hardware (carrier)/TP540xMCB.kicad_pcb (KiCad board)
At the start: 2 copper layers, 36 x 25.7 mm, 13 parts, among them J1 Input, J2 Output, J3 MountPoint, J4 MountPoint, J5 MountPoint, J6 MountPoint

Commit message: ..
Other:
- board text added: "TPS540x Carrier"
- board text removed: "TPS540x Breakout"
Changed lines of the file:
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@@
     (effects (font (size 0.9 0.9) (thickness 0.15)))
   )
-  (gr_text "TPS540x Breakout" (at 100 88.2) (layer "F.SilkS")
+  (gr_text "TPS540x Carrier" (at 100 88.2) (layer "F.SilkS")
     (effects (font (size 1 1) (thickness 0.15)))
   )
