File: Standalone Hardware (combo)/TP540xEVM.kicad_pcb (KiCad board)
At the start: 2 copper layers, 36 x 25.7 mm, 18 parts, among them J1 Input, J2 Output, U1 TPS5403

Commit message: ...
Parts:
- added J3: MountPoint, Tinker:ConnPoint, F.Cu at (90.8, 90.2)
- added J4: MountPoint, Tinker:ConnPoint, F.Cu at (109.2, 90.2)
- added J5: MountPoint, Tinker:ConnPoint, F.Cu at (90.8, 99.1)
- added J6: MountPoint, Tinker:ConnPoint, F.Cu at (109.2, 99.2)
- moved J1 0.67 mm to (86.0, 96.5)
- moved J2 0.67 mm to (114.0, 100.0)
Routing:
- net Vout: track 23.1 -> 37.9 mm
- net Vin: track 19.9 -> 26.8 mm
