File: Standalone Hardware (combo)/TP540xEVM.kicad_sch (KiCad schematic)
At the start: 13 parts, among them J1 Conn_01x01_Male, J2 Conn_01x01_Male, J3 Conn_01x01_Male, J4 Conn_01x01_Male, U1 TPS5403

Commit message: ...
Parts:
- removed J1, J2: Conn_01x01_Male, Tinker:ConnPoint, symbol Connector:Conn_01x01_Male
- added C2, C3: 330uF, Capacitor_SMD:CP_Elec_8x10, symbol Device:C_Polarized
- added J1: Input, TerminalBlock_4Ucon:TerminalBlock_4Ucon_1x02_P3.50mm_Horizontal, symbol Connector:Conn_01x02_Male
- added J2: Output, TerminalBlock_4Ucon:TerminalBlock_4Ucon_1x02_P3.50mm_Horizontal, symbol Connector:Conn_01x02_Male
- added J5, J6: MountPoint, Tinker:ConnPoint, symbol Connector:Conn_01x01_Male
- J3, J4: value Conn_01x01_Male -> MountPoint
Connections:
- net GND: now also C2.2, C3.2, J1.2 (Pin_2), J2.1 (Pin_1), J5.1 (Pin_1), J6.1 (Pin_1); no longer J3.1 (Pin_1), J4.1 (Pin_1)
- net Vin: now also J3.1 (Pin_1), C2.1, J1.1 (Pin_1)
- net Vout: now also J4.1 (Pin_1), C3.1, J2.2 (Pin_2)
