File: Module Hardware/TP540xMOD.kicad_pcb (KiCad board)
At the start: 2 copper layers, 18 x 12.2 mm, 13 parts, among them J1 Conn_01x01_Male, J2 Conn_01x01_Male, J3 Conn_01x01_Male, J4 Conn_01x01_Male, U1 TPS5403

Commit message: ...
Parts:
- added REF**: DagNabbit, Tinker:DagNabbit, B.Cu at (92.7, 95.0)
- C1, C4, C5, C6: footprint Capacitor_SMD:C_0603_1608Metric_Pad1.08x0.95mm_HandSolder -> Capacitor_SMD:C_0603_1608Metric
- R1, R2: footprint Resistor_SMD:R_0603_1608Metric_Pad0.98x0.95mm_HandSolder -> Resistor_SMD:R_0603_1608Metric
- moved L1 4.07 mm to (104.7, 95.7)
- moved D1 2.86 mm to (104.7, 90.4)
- moved J1 1.85 mm to (90.8, 90.2)
- moved J2 1.80 mm to (109.2, 90.2)
- moved C4 1.31 mm to (96.8, 98.8)
- moved C5 1.31 mm to (95.2, 98.8)
- moved C6 1.31 mm to (100.0, 98.8)
- moved R1 1.31 mm to (93.6, 98.8)
- moved R2 1.31 mm to (98.4, 98.8)
- moved J3 1.28 mm to (90.8, 99.2)
- moved J4 1.26 mm to (109.2, 99.2)
- moved U1 1.24 mm to (96.9, 94.1)
- moved C1 1.21 mm to (96.9, 90.6)
Routing:
- net Vout: track 14.1 -> 16.2 mm, vias 1 -> 0
- net Net-(R1-Pad1): track 6.53 -> 5.46 mm
- net Net-(C4-Pad1): track 7.91 -> 8.95 mm, vias 0 -> 2
- net Net-(C5-Pad1): track 3.31 -> 2.34 mm
- net Net-(C1-Pad2): track 10.8 -> 11.5 mm
- net Vin: track 5.21 -> 5.90 mm
Other:
- board size 18 x 12.2 mm -> 20.6 x 11.3 mm
- board text added: "+"
- board text added: "S. A. Miller 2024"
- board text added: "TPS540x Carrier"
- board text removed: "18.0 x 12.2"

Commit message: w00t...SMD inductor
Parts:
- L1: footprint Inductor_THT:L_Radial_D6.0mm_P4.00mm -> Tinker:IND-SMD_L7.1-W6.6
- moved L1 0.33 mm to (104.4, 95.8)
Routing:
- net GND: vias 10 -> 12
Changed lines of the file:
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@@
+    )
+  )
+  (footprint "Tinker:IND-SMD_L7.1-W6.6" (layer "F.Cu")
+    (at 104.372882 95.753077 -90)
+    (property "LCSC" "C2983095")
+    (property "Sheetfile" "TP540xMOD.kicad_sch")
+    (property "Sheetname" "")
+    (attr smd)
+    (fp_text reference "L1" (at 3.941923 2.57 180) (layer "F.SilkS")
+      (effects (font (size 0.6 0.6) (thickness 0.15)))
+    )
+    (fp_text value "L_Ferrite" (at 0 4 90) (layer "F.Fab")
+      (effects (font (size 1 1) (thickness 0.15)))
+    )
+    (fp_text user "${REFERENCE}" (at 0 0 90) (layer "F.Fab")
+      (effects (font (size 1 1) (thickness 0.15)))
+    )
+    (fp_line (start 3.3 -3.3) (end -3.3 -3.3) (layer "F.SilkS") (width 0.15))
+    (fp_line (start 3.3 -1.84) (end 3.3 -3.3) (layer "F.SilkS") (width 0.15))
+    (fp_line (start -3.3 -3.3) (end -3.3 -1.84) (layer "F.SilkS") (width 0.15))
+    (fp_line (start 3.3 3.3) (end 3.3 1.84) (layer "F.SilkS") (width 0.15))
+    (fp_line (start -3.3 1.84) (end -3.3 3.3) (layer "F.SilkS") (width 0.15))
+    (fp_line (start -3.3 3.3) (end 3.3 3.3) (layer "F.SilkS") (width 0.15))
+    (fp_circle (center -3.55 3.3) (end -3.52 3.3) (layer "F.Fab") (width 0.06) (fill none))
+    (pad "1" smd rect (at -2.91 0 270) (size 2.15 3.32) (layers "F.Cu" "F.Paste" "F.Mask")
+      (net 2 "Net-(C1-Pad2)") (pinfunction "1") (pintype "passive"))
+    (pad "2" smd rect (at 2.91 0 270) (size 2.15 3.32) (layers "F.Cu" "F.Paste" "F.Mask")
+      (net 5 "Vout") (pinfunction "2") (pintype "passive"))
+    (model "/home/tinker/Documents/LCSC-KiCAD/.3dshapes/IND-SMD_L6.6-W7.1-H3.0.wrl"
+      (offset (xyz 0.11 0 0))
+      (scale (xyz 1 1 1))
+      (rotate (xyz 0 0 0))
     )
   )
@@
     )
   )
-  (footprint "Inductor_THT:L_Radial_D6.0mm_P4.00mm" (layer "F.Cu")
-    (at 104.7 95.745 -90)
-    (descr "Inductor, Radial series, Radial, pin pitch=4.00mm, , diameter=6.0mm, http://www.abracon.com/Magnetics/radial/AIUR-07.pdf")
-    (tags "Inductor Radial series Radial pin pitch 4.00mm  diameter 6.0mm")
-    (property "Sheetfile" "TP540xMOD.kicad_sch")
-    (property "Sheetname" "")
-    (attr through_hole)
-    (fp_text reference "L1" (at 3.29 2.265) (layer "F.SilkS")
-      (effects (font (size 0.6 0.6) (thickness 0.15)))
-    )
-    (fp_text value "L_Ferrite" (at 0 5.08 90) (layer "F.Fab")
-      (effects (font (size 1 1) (thickness 0.15)))
-    )
-    (fp_text user "${REFERENCE}" (at 0 -5.08 90) (layer "F.Fab")
-      (effects (font (size 1 1) (thickness 0.15)))
-    )
-    (fp_arc (start 2.85426 1.26) (mid 0 3.12) (end -2.85426 1.26) (layer "F.SilkS") (width 0.12))
-    (fp_arc (start -2.85426 -1.26) (mid 0 -3.12) (end 2.85426 -1.26) (layer "F.SilkS") (width 0.12))
-    (fp_circle (center 0 0) (end 4 0) (layer "F.CrtYd") (width 0.05) (fill none))
-    (fp_circle (center 0 0) (end 3 0) (layer "F.Fab") (width 0.1) (fill none))
-    (pad "1" thru_hole circle (at -2.5 0 270) (size 2 2) (drill 1) (layers *.Cu *.Mask)
-      (net 2 "Net-(C1-Pad2)") (pinfunction "1") (pintype "passive"))
-    (pad "2" thru_hole circle (at 2.5 0 270) (size 2 2) (drill 1) (layers *.Cu *.Mask)
-      (net 5 "Vout") (pinfunction "2") (pintype "passive"))
-    (model "${KICAD6_3DMODEL_DIR}/Inductor_THT.3dshapes/L_Radial_D6.0mm_P4.00mm.wrl"
-      (offset (xyz -2 0 0))
-      (scale (xyz 1 1 1))
-      (rotate (xyz 0 0 0))
-    )
-  )
   (footprint "Capacitor_SMD:C_0603_1608Metric" (layer "F.Cu")
     (at 100 98.825 90)
@@
     (property "Sheetname" "")
     (attr through_hole)
-    (fp_text reference "J4" (at 0 -1.27) (layer "F.SilkS")
+    (fp_text reference "J4" (at -1.8 0.4) (layer "F.SilkS")
       (effects (font (size 0.6 0.6) (thickness 0.15)))
     )
@@
     (property "Sheetname" "")
     (attr through_hole)
-    (fp_text reference "J3" (at 0 -1.27) (layer "F.SilkS")
+    (fp_text reference "J3" (at 1.8 0.4) (layer "F.SilkS")
       (effects (font (size 0.6 0.6) (thickness 0.15)))
     )
@@
     (property "Sheetname" "")
     (attr through_hole)
-    (fp_text reference "J2" (at 0 1.33) (layer "F.SilkS")
+    (fp_text reference "J2" (at -1.8 -0.2) (layer "F.SilkS")
       (effects (font (size 0.6 0.6) (thickness 0.15)))
     )
@@
     (property "Sheetname" "")
     (attr through_hole)
-    (fp_text reference "J1" (at 0 1.33) (layer "F.SilkS")
+    (fp_text reference "J1" (at 1.8 -0.2) (layer "F.SilkS")
       (effects (font (size 0.6 0.6) (thickness 0.15)))
     )
@@
     (effects (font (size 0.75 0.75) (thickness 0.15)) (justify mirror))
   )
-  (gr_text "+" (at 107.5 90.17) (layer "F.SilkS")
+  (gr_text "+" (at 109.22 91.44) (layer "F.SilkS")
     (effects (font (size 0.9 0.9) (thickness 0.15)))
   )
-  (gr_text "G" (at 92.5 99.2) (layer "F.SilkS")
+  (gr_text "G" (at 90.805 97.79) (layer "F.SilkS")
     (effects (font (size 0.9 0.9) (thickness 0.15)))
   )
-  (gr_text "G" (at 107.5 99.2) (layer "F.SilkS")
+  (gr_text "G" (at 109.22 97.79) (layer "F.SilkS")
     (effects (font (size 0.9 0.9) (thickness 0.15)))
   )
@@
     (effects (font (size 1 1) (thickness 0.15)))
   )
-  (gr_text "+" (at 92.5 90.17) (layer "F.SilkS")
+  (gr_text "+" (at 90.805 91.44) (layer "F.SilkS")
     (effects (font (size 0.9 0.9) (thickness 0.15)))
   )
@@
   (segment (start 96.75 99.65) (end 96.8 99.6) (width 0.25) (layer "F.Cu") (net 4))
   (segment (start 93.6 99.65) (end 96.75 99.65) (width 0.25) (layer "F.Cu") (net 4))
+  (via (at 100.33 90.805) (size 0.8) (drill 0.4) (layers "F.Cu" "B.Cu") (free) (net 4))
   (via (at 96.2217 94.78) (size 0.8) (drill 0.4) (layers "F.Cu" "B.Cu") (free) (net 4))
+  (via (at 93.345 90.805) (size 0.8) (drill 0.4) (layers "F.Cu" "B.Cu") (free) (net 4))
   (via (at 97.4917 93.51) (size 0.8) (drill 0.4) (layers "F.Cu" "B.Cu") (free) (net 4))
   (via (at 96.2217 93.51) (size 0.8) (drill 0.4) (layers "F.Cu" "B.Cu") (free) (net 4))
@@
     (polygon
       (pts
-        (xy 118.4467 113.22)
-        (xy 81.6167 113.22)
-        (xy 81.6167 86.55)
-        (xy 118.4467 86.55)
+        (xy 110.8267 101.155)
+        (xy 89.2367 101.155)
+        (xy 89.2367 88.455)
+        (xy 110.8267 88.455)
       )
     )
@@
     (polygon
       (pts
-        (xy 118.4467 113.22)
-        (xy 81.6167 113.22)
-        (xy 81.6167 86.55)
-        (xy 118.4467 86.55)
+        (xy 110.8267 101.155)
+        (xy 89.2367 101.155)
+        (xy 89.2367 88.455)
+        (xy 110.8267 88.455)
       )
     )
