File: Module Hardware/TP540xMOD.kicad_pcb (KiCad board)
At the start: 2 copper layers, 20.6 x 11.3 mm, 14 parts, among them J1 Conn_01x01_Male, J2 Conn_01x01_Male, J3 Conn_01x01_Male, J4 Conn_01x01_Male, U1 TPS5403

Commit message: Some cleanup...
Parts:
- added G***: LOGO, Tinker:NerdMage, B.Cu at (102.9, 96.5)
