File: Module Hardware/TP540xMOD.kicad_sch (KiCad schematic)
At the start: 13 parts, among them J1 Conn_01x01_Male, J2 Conn_01x01_Male, J3 Conn_01x01_Male, J4 Conn_01x01_Male, U1 TPS5403

Commit message: w00t...SMD inductor
Parts:
- L1: footprint Inductor_THT:L_Radial_D6.0mm_P4.00mm -> Tinker:IND-SMD_L7.1-W6.6; LCSC (none) -> C2983095
Changed lines of the file:
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@@
+    (stroke (width 0) (type default) (color 0 0 0 0))
+  )
+  (wire (pts (xy 185.42 93.98) (xy 185.42 107.95))
     (stroke (width 0) (type default) (color 0 0 0 0))
   )
@@
   )
   (wire (pts (xy 124.46 99.06) (xy 124.46 100.33))
-    (stroke (width 0) (type default) (color 0 0 0 0))
-  )
-  (wire (pts (xy 185.42 107.95) (xy 185.42 93.98))
     (stroke (width 0) (type default) (color 0 0 0 0))
   )
@@
     (property "Reference" "L1" (id 0) (at 181.61 87.63 90))
     (property "Value" "L_Ferrite" (id 1) (at 181.61 90.17 90))
-    (property "Footprint" "Inductor_THT:L_Radial_D6.0mm_P4.00mm" (id 2) (at 181.61 93.98 0)
+    (property "Footprint" "Tinker:IND-SMD_L7.1-W6.6" (id 2) (at 181.61 93.98 0)
       (effects (font (size 1.27 1.27)) hide)
     )
     (property "Datasheet" "~" (id 3) (at 181.61 93.98 0)
+      (effects (font (size 1.27 1.27)) hide)
+    )
+    (property "LCSC" "C2983095" (id 4) (at 181.61 93.98 90)
       (effects (font (size 1.27 1.27)) hide)
     )
@@
       (reference "J4") (unit 1) (value "Conn_01x01_Male") (footprint "Tinker:ConnPoint")
     )
-    (path "/479f3f0b-5f70-458d-a591-f099cd39a0d2"
-      (reference "L1") (unit 1) (value "L_Ferrite") (footprint "Inductor_THT:L_Radial_D6.0mm_P4.00mm")
+    (path "/27aff825-147f-432a-9901-657a935859c3"
+      (reference "L1") (unit 1) (value "L_Ferrite") (footprint "Tinker:IND-SMD_L7.1-W6.6")
     )
     (path "/794b9bb4-29b7-450a-bb76-0318a7f3d068"
