File: Carrier Hardware/TP540xMCB.kicad_pcb (KiCad board)
At the start: 2 copper layers, 36 x 25.7 mm, 10 parts, among them J1 Input, J2 Output

Commit message: Some cleanup...
Parts:
- added G***: LOGO, Tinker:NerdMage, F.Cu at (100.3, 97.2)
